File: CameraSlider/CameraSliderV1.brd (EAGLE design)
At the start: 50 x 80 mm, 41 parts, among them SW1 ROTARTY_ENCODER, U3 ATMEGA328P_TQFP, Y2 16MHz

Commit message: Updated cameraslider
Parts:
- moved U$15 13.0 mm to (11.5, 13.6)
- moved R7 11.8 mm to (21.4, 26.4), turned to 0 degrees
- moved R8 3.39 mm to (17.0, 26.3), turned to 180 degrees
Routing:
- net SCL: track 44.0 -> 40.5 mm
- net SDA: track 36.5 -> 34.6 mm
- net VCC: track 291.2 -> 292.8 mm
Changed lines of the file:
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@@
 <element name="S4" library="SparkFun" package="TACTILE_SWITCH_SMD" value="RST" x="15.4178" y="36.9316" rot="R270"/>
 <element name="U$1" library="RobThePyro" package="A4988MOD" value="A4988MOD" x="30.7594" y="66.421" rot="R90"/>
-<element name="U$15" library="RobThePyro" package="SHROOM" value="SHROOM5MM" x="0.5334" y="6.5786"/>
+<element name="U$15" library="RobThePyro" package="SHROOM" value="SHROOM5MM" x="11.4554" y="13.589"/>
 <element name="U$2" library="RobThePyro" package="D-SUN_MP1584" value="" x="9.652" y="52.0954" rot="R270"/>
 <element name="U3" library="SparkFun-DigitalIC" package="TQFP32-08" value="ATMEGA328P_TQFP" x="36.957" y="42.7736" rot="R225">
@@
 </element>
 <element name="I2C" library="pinhead" package="1X04" value="" x="16.6624" y="29.3116"/>
-<element name="R7" library="resistor" package="M0805" value="4k7" x="9.8552" y="28.956" rot="R90"/>
-<element name="R8" library="resistor" package="M0805" value="4k7" x="20.32" y="25.6794"/>
+<element name="R7" library="resistor" package="M0805" value="4k7" x="21.3868" y="26.3652"/>
+<element name="R8" library="resistor" package="M0805" value="4k7" x="16.9926" y="26.3398" rot="R180"/>
 <element name="USART" library="pinhead" package="1X04" value="" x="23.9014" y="2.9972"/>
 <element name="ENC" library="pinhead" package="1X05" value="" x="42.6896" y="20.3316"/>
@@
 <wire x1="10.0308" y1="32.8574" x2="10.3632" y2="32.8574" width="0.8128" layer="1"/>
 <wire x1="10.3632" y1="32.8574" x2="12.761" y2="32.893" width="0.8128" layer="1"/>
-<wire x1="12.761" y1="32.893" x2="20.1422" y2="32.893" width="0.8128" layer="1"/>
-<wire x1="20.1422" y1="32.893" x2="25.1206" y2="32.893" width="0.8128" layer="1"/>
+<wire x1="12.761" y1="32.893" x2="15.7988" y2="32.893" width="0.8128" layer="1"/>
+<wire x1="15.7988" y1="32.893" x2="25.1206" y2="32.893" width="0.8128" layer="1"/>
 <wire x1="32.507459375" y1="41.152484375" x2="36.516175" y2="45.1612" width="0.4064" layer="1"/>
 <wire x1="36.516175" y1="45.1612" x2="37.6682" y2="45.1612" width="0.4064" layer="1"/>
@@
 <wire x1="7.44" y1="32.8574" x2="9.5758" y2="32.8574" width="0.8128" layer="1"/>
 <wire x1="9.5758" y1="32.8574" x2="10.3632" y2="32.8574" width="0.8128" layer="1"/>
-<wire x1="9.8552" y1="29.906" x2="9.8552" y2="32.578" width="0.4064" layer="1"/>
 <wire x1="9.8552" y1="32.578" x2="9.5758" y2="32.8574" width="0.4064" layer="1"/>
-<wire x1="21.27" y1="25.6794" x2="21.27" y2="27.9552" width="0.4064" layer="1"/>
-<wire x1="20.1422" y1="29.0322" x2="20.1422" y2="32.893" width="0.4064" layer="1"/>
 <contactref element="JP1" pad="5"/>
 <contactref element="JP1" pad="6"/>
@@
 <wire x1="30.9626" y1="0.4318" x2="30.607" y2="0.7874" width="0.6096" layer="1"/>
 <contactref element="I2C" pad="2"/>
-<wire x1="20.1422" y1="29.0322" x2="21.27" y2="27.9552" width="0" layer="19" extent="1-1"/>
-<wire x1="15.3924" y1="29.3116" x2="12.761" y2="32.893" width="0" layer="19" extent="1-1"/>
+<wire x1="16.0426" y1="26.3398" x2="16.0426" y2="26.6548" width="0.6096" layer="1"/>
+<wire x1="16.0426" y1="26.6548" x2="15.4178" y2="27.2796" width="0.6096" layer="1"/>
+<wire x1="15.4178" y1="27.2796" x2="15.4178" y2="29.2862" width="0.6096" layer="1"/>
+<wire x1="15.4178" y1="29.2862" x2="15.3924" y2="29.3116" width="0.6096" layer="1"/>
+<wire x1="15.3924" y1="29.3116" x2="15.3924" y2="32.4866" width="0.6096" layer="1"/>
+<wire x1="15.3924" y1="32.4866" x2="15.7988" y2="32.893" width="0.6096" layer="1"/>
+<wire x1="22.3368" y1="26.3652" x2="23.9928" y2="26.3652" width="0.6096" layer="1"/>
+<wire x1="23.9928" y1="26.3652" x2="25.2374" y2="27.6098" width="0.6096" layer="1"/>
 </signal>
 <signal name="MISO">
@@
 <wire x1="40.1574" y1="37.8714" x2="40.1574" y2="33.4772" width="0.6096" layer="1"/>
 <wire x1="40.1574" y1="33.4772" x2="30.2768" y2="23.5966" width="0.6096" layer="1"/>
-<wire x1="30.2768" y1="23.5966" x2="18.7706" y2="23.5966" width="0.6096" layer="1"/>
-<wire x1="18.7706" y1="23.5966" x2="15.113" y2="27.2542" width="0.6096" layer="1"/>
 <contactref element="R7" pad="1"/>
 <contactref element="I2C" pad="4"/>
-<wire x1="15.113" y1="27.2542" x2="20.4724" y2="29.3116" width="0" layer="19" extent="1-1"/>
-<wire x1="9.8552" y1="28.006" x2="15.113" y2="27.2542" width="0" layer="19" extent="1-1"/>
+<wire x1="30.2768" y1="23.5966" x2="21.7424" y2="23.5966" width="0.6096" layer="1"/>
+<wire x1="21.7424" y1="23.5966" x2="20.447" y2="24.892" width="0.6096" layer="1"/>
+<wire x1="20.447" y1="24.892" x2="20.447" y2="26.355" width="0.6096" layer="1"/>
+<wire x1="20.447" y1="26.355" x2="20.4368" y2="26.3652" width="0.6096" layer="1"/>
+<wire x1="20.4368" y1="26.3652" x2="20.4368" y2="29.276" width="0.6096" layer="1"/>
+<wire x1="20.4368" y1="29.276" x2="20.4724" y2="29.3116" width="0.6096" layer="1"/>
 </signal>
 <signal name="SCL">
 <contactref element="U3" pad="28"/>
-<wire x1="30.6324" y1="22.4028" x2="17.2466" y2="22.4028" width="0.6096" layer="1"/>
-<wire x1="17.2466" y1="22.4028" x2="12.573" y2="27.0764" width="0.6096" layer="1"/>
 <wire x1="39.70948125" y1="39.455428125" x2="39.741771875" y2="39.455428125" width="0.4064" layer="1"/>
 <wire x1="39.741771875" y1="39.455428125" x2="41.3258" y2="37.8714" width="0.4064" layer="1"/>
 <wire x1="41.3258" y1="37.8714" x2="41.3258" y2="33.0962" width="0.6096" layer="1"/>
 <wire x1="41.3258" y1="33.0962" x2="30.6324" y2="22.4028" width="0.6096" layer="1"/>
-<wire x1="12.573" y1="27.0764" x2="10.7848" y2="27.0764" width="0.4064" layer="1"/>
 <contactref element="R8" pad="1"/>
 <contactref element="I2C" pad="3"/>
-<wire x1="19.37" y1="25.6794" x2="17.9324" y2="29.3116" width="0" layer="19" extent="1-1"/>
-<wire x1="17.2466" y1="22.4028" x2="19.37" y2="25.6794" width="0" layer="19" extent="1-1"/>
+<wire x1="30.6324" y1="22.4028" x2="20.066" y2="22.4028" width="0.6096" layer="1"/>
+<wire x1="20.066" y1="22.4028" x2="17.9324" y2="24.5364" width="0.6096" layer="1"/>
+<wire x1="17.9324" y1="24.5364" x2="17.9324" y2="26.3296" width="0.6096" layer="1"/>
+<wire x1="17.9324" y1="26.3296" x2="17.9426" y2="26.3398" width="0.6096" layer="1"/>
+<wire x1="17.9426" y1="26.3398" x2="17.9426" y2="29.3014" width="0.6096" layer="1"/>
+<wire x1="17.9426" y1="29.3014" x2="17.9324" y2="29.3116" width="0.6096" layer="1"/>
 </signal>
 <signal name="ENC_A">
