File: LoRa1278 Breakout/LoRa1278_Breakout.brd (EAGLE design)
At the start: 35.2 x 24.8 mm, 9 parts, among them IC1 REG1117

Commit message: Working on constant current load :)
Parts:
- added JP2: (no value), pinhead:1X01
- added U$2: SHROOM5MM, RobThePyro:SHROOM
Connections:
- net +3V3: now also IC1.4
- net N$11: now also JP2.1
Routing:
- net N$11: track 9.97 -> 12.9 mm
- net N$20: track 0.00 -> 2.00 mm
- net N$19: track 0.00 -> 2.00 mm
- net N$18: track 0.00 -> 2.00 mm
- net N$17: track 0.00 -> 2.00 mm
- net N$16: track 0.00 -> 2.00 mm
- net N$15: track 0.00 -> 2.00 mm
- net N$14: track 0.00 -> 2.00 mm
- net N$13: track 0.00 -> 2.00 mm
- added copper zone on layer 1, net +3V3
Other:
- board size 35.2 x 24.8 mm -> 35 x 25 mm
- board text added: "LoRa1278 Breakout"
Changed lines of the file:
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@@
 <board>
 <plain>
-<wire x1="0" y1="0" x2="35.23" y2="0" width="0" layer="20"/>
-<wire x1="35.23" y1="0" x2="35.23" y2="24.755" width="0" layer="20"/>
-<wire x1="35.23" y1="24.755" x2="0" y2="24.755" width="0" layer="20"/>
-<wire x1="0" y1="24.755" x2="0" y2="0" width="0" layer="20"/>
+<text x="15.875" y="19.05" size="2.032" layer="1" ratio="15">LoRa1278
+Breakout</text>
+<wire x1="0" y1="0" x2="0" y2="25" width="0" layer="20"/>
+<wire x1="0" y1="25" x2="35" y2="25" width="0" layer="20"/>
+<wire x1="35" y1="25" x2="35" y2="0" width="0" layer="20"/>
+<wire x1="35" y1="0" x2="0" y2="0" width="0" layer="20"/>
 </plain>
 <attributes>
@@
 <element name="U$1" library="NiceRF" package="LORA1278" value="LORA1278-433" x="18.415" y="15.24" rot="R90"/>
 <element name="JP1" library="pinhead" package="1X13" value="" x="16.51" y="1.27"/>
+<element name="U$2" library="RobThePyro" package="SHROOM" value="SHROOM5MM" x="11.43" y="14.605"/>
+<element name="JP2" library="pinhead" package="1X01" value="" x="8" y="23"/>
 </elements>
 <signals>
@@
 <wire x1="8.2296" y1="11.0744" x2="28.4394" y2="11.0744" width="0.6096" layer="1"/>
 <wire x1="28.4394" y1="11.0744" x2="28.575" y2="11.21" width="0.6096" layer="1"/>
-<wire x1="9.525" y1="18.415" x2="8.2296" y2="11.0744" width="0" layer="19" extent="1-1"/>
-<wire x1="2.54" y1="18.415" x2="2.54" y2="18.415" width="0" layer="19" extent="1-16"/>
-<wire x1="2.54" y1="23.495" x2="2.54" y2="18.415" width="0" layer="19" extent="1-1"/>
-<wire x1="2.54" y1="23.495" x2="2.54" y2="23.495" width="0" layer="19" extent="1-16"/>
 <wire x1="28.575" y1="11.21" x2="28.575" y2="16.02" width="0.6096" layer="1"/>
 <wire x1="28.575" y1="16.02" x2="29.065" y2="16.51" width="0.6096" layer="1"/>
 <wire x1="30.8" y1="11.43" x2="28.795" y2="11.43" width="0.6096" layer="1"/>
 <wire x1="28.795" y1="11.43" x2="28.575" y2="11.21" width="0.6096" layer="1"/>
+<wire x1="2.54" y1="23.495" x2="2.54" y2="23.495" width="0" layer="19" extent="1-16"/>
+<wire x1="2.54" y1="18.415" x2="2.54" y2="23.495" width="0" layer="19" extent="1-16"/>
+<wire x1="2.54" y1="18.415" x2="2.54" y2="18.415" width="0" layer="19" extent="1-16"/>
+<wire x1="8.2296" y1="11.0744" x2="9.525" y2="18.415" width="0" layer="19" extent="1-1"/>
 </signal>
 <signal name="VCC">
@@
 <wire x1="32.7" y1="8.89" x2="32.7" y2="7.935" width="0.6096" layer="1"/>
 <wire x1="32.7" y1="7.935" x2="29.845" y2="5.08" width="0.6096" layer="1"/>
+<contactref element="IC1" pad="4"/>
+<polygon width="0.4064" layer="1">
+<vertex x="0.635" y="6.35"/>
+<vertex x="0.635" y="16.51"/>
+<vertex x="3.81" y="16.51"/>
+<vertex x="3.81" y="9.525"/>
+</polygon>
+<wire x1="1.9304" y1="13.335" x2="8.2296" y2="13.3604" width="0" layer="19" extent="1-1"/>
 </signal>
 <signal name="N$11">
@@
 <contactref element="J$1" pad="SIG"/>
 <wire x1="2.54" y1="20.955" x2="8.89" y2="20.955" width="0.6096" layer="1"/>
-<wire x1="8.89" y1="20.955" x2="10.795" y2="22.86" width="0.6096" layer="1"/>
+<wire x1="8.89" y1="20.955" x2="10.4675" y2="22.5325" width="0.6096" layer="1"/>
+<wire x1="10.4675" y1="22.5325" x2="10.795" y2="22.86" width="0.6096" layer="1"/>
 <wire x1="10.795" y1="22.86" x2="10.795" y2="22.8854" width="0.6096" layer="1"/>
 <wire x1="10.795" y1="22.8854" x2="10.8966" y2="22.987" width="0.6096" layer="1"/>
 <wire x1="10.8966" y1="22.987" x2="10.8966" y2="23.7216" width="0.6096" layer="1"/>
 <wire x1="10.8966" y1="23.7216" x2="10.915" y2="23.74" width="0.6096" layer="1"/>
+<contactref element="JP2" pad="1"/>
+<wire x1="8" y1="23" x2="10.4675" y2="23" width="0.6096" layer="1"/>
+<wire x1="10.4675" y1="23" x2="10.4675" y2="22.5325" width="0.6096" layer="1"/>
 </signal>
 <signal name="N$12">
@@
 <wire x1="29.21" y1="1.905" x2="29.21" y2="1.27" width="0.4064" layer="1"/>
 </signal>
+<signal name="N$13">
+<wire x1="0" y1="24" x2="0" y2="26" width="0.4064" layer="1"/>
+</signal>
+<signal name="N$14">
+<wire x1="-1" y1="25" x2="1" y2="25" width="0.4064" layer="1"/>
+</signal>
+<signal name="N$15">
+<wire x1="34" y1="25" x2="36" y2="25" width="0.4064" layer="1"/>
+</signal>
+<signal name="N$16">
+<wire x1="35" y1="26" x2="35" y2="24" width="0.4064" layer="1"/>
+</signal>
+<signal name="N$17">
+<wire x1="34" y1="0" x2="36" y2="0" width="0.4064" layer="1"/>
+</signal>
+<signal name="N$18">
+<wire x1="35" y1="-1" x2="35" y2="1" width="0.4064" layer="1"/>
+</signal>
+<signal name="N$19">
+<wire x1="0" y1="-1" x2="0" y2="1" width="0.4064" layer="1"/>
+</signal>
+<signal name="N$20">
+<wire x1="-1" y1="0" x2="1" y2="0" width="0.4064" layer="1"/>
+</signal>
 </signals>
 </board>
 </drawing>
+<compatibility>
+<note version="6.3" minversion="6.2.2" severity="warning">
+Since Version 6.2.2 text objects can contain more than one line,
+which will not be processed correctly with this version.
+</note>
+</compatibility>
 </eagle>
