File: LoRa1278 Breakout/LoRa1278_Breakout.sch (EAGLE design)
At the start: 9 parts, among them IC1 REG1117

Commit message: Working on constant current load :)
Parts:
- added JP2: (no value), pinhead:PINHD-1X1
- added U$2: SHROOM5MM, RobThePyro:SHROOM5MM
Connections:
- net +3V3: now also IC1.$VOUT
- net N$11: now also JP2.1
Changed lines of the file:
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@@
 <part name="R1" library="resistor" deviceset="R-US_" device="R0805"/>
 <part name="JP1" library="pinhead" deviceset="PINHD-1X13" device=""/>
+<part name="U$2" library="RobThePyro" deviceset="SHROOM" device="5MM"/>
+<part name="JP2" library="pinhead" deviceset="PINHD-1X1" device=""/>
 </parts>
 <sheets>
@@
 <instance part="R1" gate="G$1" x="38.1" y="81.28" rot="R180"/>
 <instance part="JP1" gate="A" x="-101.6" y="10.16" rot="MR0"/>
+<instance part="U$2" gate="G$1" x="-66.04" y="55.88"/>
+<instance part="JP2" gate="G$1" x="27.94" y="22.86" rot="R90"/>
 </instances>
 <busses>
@@
 <wire x1="30.48" y1="81.28" x2="30.48" y2="86.36" width="0.1524" layer="91"/>
 <junction x="30.48" y="86.36"/>
+<pinref part="IC1" gate="G$1" pin="$VOUT"/>
+<wire x1="10.16" y1="83.82" x2="10.16" y2="86.36" width="0.1524" layer="91"/>
+<junction x="10.16" y="86.36"/>
 </segment>
 <segment>
@@
 <pinref part="U$1" gate="G$1" pin="ANT"/>
 <pinref part="J$1" gate="1" pin="SIGNAL"/>
-<wire x1="20.32" y1="12.7" x2="33.02" y2="12.7" width="0.1524" layer="91"/>
+<wire x1="20.32" y1="12.7" x2="27.94" y2="12.7" width="0.1524" layer="91"/>
+<pinref part="JP2" gate="G$1" pin="1"/>
+<wire x1="27.94" y1="12.7" x2="33.02" y2="12.7" width="0.1524" layer="91"/>
+<wire x1="27.94" y1="20.32" x2="27.94" y2="12.7" width="0.1524" layer="91"/>
+<junction x="27.94" y="12.7"/>
 </segment>
 </net>
