File: RAMPS_UPS/RAMPS_UPS.brd (EAGLE design)
At the start: 50 x 50 mm, 6 parts, among them Q1 BSO201SP, Q2 BSO201SP, Q3 BSO201SP, X1 MSTBA4, X2 MSTBA4, X3 MSTBA2

Commit message: Updates...
Parts:
- added C1: 220nF, resistor:C0805K
- added C2: (no value), resistor:PANASONIC_C
- added C3: (no value), resistor:PANASONIC_G
- added D1: (no value), diode:SMB
- added L1: DR125, inductors:DR125
- added R1: 1.15k, resistor:R0805
- added R2: 1.5k, resistor:R0805
- added R3: 15.4k, resistor:R0805
- added U1: LM2585S-ADJ, NSC_By_element14_Batch_1.1:TO170P1435X457-5N
Connections:
- new net +12V: C2.+, L1.1, U1.5
- new net N$2: R2.1, R3.2, U1.2
- new net N$3: R1.2, U1.1
- new net N$4: C1.1, R1.1
- new net N$7: D1.A, L1.2, U1.4
- new net N$8: C3.+, D1.C
- net GND: now also C1.2, C2.-, C3.-, R2.2, U1.3, U1.6
Changed lines of the file:
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@@
 <layer number="97" name="Info" color="7" fill="1" visible="no" active="no"/>
 <layer number="98" name="Guide" color="6" fill="1" visible="no" active="no"/>
+<layer number="99" name="SpiceOrder" color="5" fill="1" visible="no" active="no"/>
 </layers>
 <board>
@@
 <element name="Q2" library="transistor-fet" package="SO-8" value="BSO201SP" x="46.355" y="17.145" rot="R90"/>
 <element name="Q3" library="transistor-fet" package="SO-8" value="BSO201SP" x="46.355" y="24.765" rot="R270"/>
+<element name="U1" library="NSC_By_element14_Batch_1.1" package="TO170P1435X457-5N" value="LM2585S-ADJ" x="8.255" y="43.815">
+<attribute name="OC_FARNELL" value="1469182" x="8.255" y="43.815" size="1.778" layer="27" display="off"/>
+<attribute name="SUPPLIER" value="National Semiconductor" x="8.255" y="43.815" size="1.778" layer="27" display="off"/>
+<attribute name="MPN" value="LM2585S-ADJ" x="8.255" y="43.815" size="1.778" layer="27" display="off"/>
+<attribute name="OC_NEWARK" value="41K3722" x="8.255" y="43.815" size="1.778" layer="27" display="off"/>
+<attribute name="PACKAGE" value="TO-263-5" x="8.255" y="43.815" size="1.778" layer="27" display="off"/>
+</element>
+<element name="R1" library="resistor" package="R0805" value="1.15k" x="5.08" y="27.94" rot="R90"/>
+<element name="R2" library="resistor" package="R0805" value="1.5k" x="7.62" y="24.765"/>
+<element name="R3" library="resistor" package="R0805" value="15.4k" x="13.335" y="20.32"/>
+<element name="C1" library="resistor" package="C0805K" value="220nF" x="10.795" y="29.21"/>
+<element name="C2" library="resistor" package="PANASONIC_C" value="" x="19.685" y="30.48"/>
+<element name="C3" library="resistor" package="PANASONIC_G" value="" x="25.4" y="43.815"/>
+<element name="D1" library="diode" package="SMB" value="" x="18.415" y="35.56" rot="R180"/>
+<element name="L1" library="inductors" package="DR125" value="DR125" x="31.115" y="31.115"/>
 </elements>
 <signals>
@@
 </polygon>
 <contactref element="X3" pad="1"/>
+<contactref element="R2" pad="2"/>
+<contactref element="U1" pad="6"/>
+<contactref element="U1" pad="3"/>
+<contactref element="C1" pad="2"/>
+<contactref element="C2" pad="-"/>
+<contactref element="C3" pad="-"/>
+<wire x1="46.355" y1="10.16" x2="46.355" y2="40.005" width="0" layer="19" extent="1-1"/>
+<wire x1="36.195" y1="10.16" x2="46.355" y2="10.16" width="0" layer="19" extent="1-1"/>
+<wire x1="19.05" y1="10.16" x2="36.195" y2="10.16" width="0" layer="19" extent="1-1"/>
+<wire x1="8.89" y1="10.16" x2="19.05" y2="10.16" width="0" layer="19" extent="1-1"/>
+<wire x1="8.255" y1="43.9674" x2="8.89" y2="10.16" width="0" layer="19" extent="1-1"/>
+<wire x1="8.255" y1="34.7726" x2="8.255" y2="43.9674" width="0" layer="19" extent="1-1"/>
+<wire x1="8.57" y1="24.765" x2="8.255" y2="34.7726" width="0" layer="19" extent="1-1"/>
+<wire x1="11.795" y1="29.21" x2="8.57" y2="24.765" width="0" layer="19" extent="1-1"/>
+<wire x1="17.635" y1="30.48" x2="11.795" y2="29.21" width="0" layer="19" extent="1-1"/>
+<wire x1="21.15" y1="43.815" x2="17.635" y2="30.48" width="0" layer="19" extent="1-1"/>
 </signal>
 <signal name="V+">
@@
 <wire x1="41.275" y1="15.24" x2="41.275" y2="14.4018" width="1.016" layer="1"/>
 </signal>
+<signal name="N$2">
+<contactref element="R3" pad="2"/>
+<contactref element="R2" pad="1"/>
+<contactref element="U1" pad="2"/>
+<wire x1="6.67" y1="24.765" x2="14.285" y2="20.32" width="0" layer="19" extent="1-1"/>
+<wire x1="6.5532" y1="34.7726" x2="6.67" y2="24.765" width="0" layer="19" extent="1-1"/>
+</signal>
+<signal name="N$3">
+<contactref element="U1" pad="1"/>
+<contactref element="R1" pad="2"/>
+<wire x1="4.8514" y1="34.7726" x2="5.08" y2="28.89" width="0" layer="19" extent="1-1"/>
+</signal>
+<signal name="N$4">
+<contactref element="R1" pad="1"/>
+<contactref element="C1" pad="1"/>
+<wire x1="5.08" y1="26.99" x2="9.795" y2="29.21" width="0" layer="19" extent="1-1"/>
+</signal>
+<signal name="N$8">
+<contactref element="C3" pad="+"/>
+<contactref element="D1" pad="C"/>
+<wire x1="29.65" y1="43.815" x2="20.615" y2="35.56" width="0" layer="19" extent="1-1"/>
+</signal>
+<signal name="+12V">
+<contactref element="C2" pad="+"/>
+<contactref element="U1" pad="5"/>
+<contactref element="L1" pad="1"/>
+<wire x1="21.735" y1="30.48" x2="26.14" y2="31.115" width="0" layer="19" extent="1-1"/>
+<wire x1="11.6586" y1="34.7726" x2="21.735" y2="30.48" width="0" layer="19" extent="1-1"/>
+</signal>
+<signal name="N$7">
+<contactref element="U1" pad="4"/>
+<contactref element="D1" pad="A"/>
+<contactref element="L1" pad="2"/>
+<wire x1="16.215" y1="35.56" x2="36.09" y2="31.115" width="0" layer="19" extent="1-1"/>
+<wire x1="9.9568" y1="34.7726" x2="16.215" y2="35.56" width="0" layer="19" extent="1-1"/>
+</signal>
 </signals>
