File: RAMPS_UPS/RAMPS_UPS.sch (EAGLE design)
At the start: 6 parts, among them Q1 BSO201SP, Q2 BSO201SP, Q3 BSO201SP, X1 MSTBA4, X2 MSTBA4, X3 MSTBA2

Commit message: Updates...
Parts:
- added C1: 220nF, resistor:C-USC0805K
- added C2: (no value), resistor:CPOL-USC
- added C3: (no value), resistor:CPOL-USG
- added D1: (no value), diode:DIODE-SMB
- added L1: DR125, inductors:DR125
- added R1: 1.15k, resistor:R-US_R0805
- added R2: 1.5k, resistor:R-US_R0805
- added R3: 15.4k, resistor:R-US_R0805
- added U1: LM2585S-ADJ, NSC_By_element14_Batch_1.1:LM2585S-ADJ
Connections:
- new net +12V: C2.+, L1.1, U1.VIN
- new net N$2: R2.1, R3.2, U1.FB
- new net N$3: R1.2, U1.COMP
- new net N$4: C1.1, R1.1
- new net N$7: D1.A, L1.2, U1.SW
- new net N$8: C3.+, D1.C
- net GND: now also C1.2, C2.-, C3.-, R2.2, U1.GND, U1.GND_2
Changed lines of the file:
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@@
 <layer number="97" name="Info" color="7" fill="1" visible="yes" active="yes"/>
 <layer number="98" name="Guide" color="6" fill="1" visible="yes" active="yes"/>
+<layer number="99" name="SpiceOrder" color="5" fill="1" visible="yes" active="yes"/>
 </layers>
 <schematic xreflabel="%F%N/%S.%C%R" xrefpart="/%S.%C%R">
@@
 <part name="Q2" library="transistor-fet" deviceset="BSO201SP" device=""/>
 <part name="Q3" library="transistor-fet" deviceset="BSO201SP" device=""/>
+<part name="U1" library="NSC_By_element14_Batch_1.1" deviceset="LM2585S-ADJ" device=""/>
+<part name="R1" library="resistor" deviceset="R-US_" device="R0805" value="1.15k"/>
+<part name="R2" library="resistor" deviceset="R-US_" device="R0805" value="1.5k"/>
+<part name="R3" library="resistor" deviceset="R-US_" device="R0805" value="15.4k"/>
+<part name="C1" library="resistor" deviceset="C-US" device="C0805K" value="220nF"/>
+<part name="GND6" library="supply1" deviceset="GND" device=""/>
+<part name="GND7" library="supply1" deviceset="GND" device=""/>
+<part name="GND8" library="supply1" deviceset="GND" device=""/>
+<part name="C2" library="resistor" deviceset="CPOL-US" device="C"/>
+<part name="C3" library="resistor" deviceset="CPOL-US" device="G"/>
+<part name="GND9" library="supply1" deviceset="GND" device=""/>
+<part name="GND10" library="supply1" deviceset="GND" device=""/>
+<part name="P+9" library="supply1" deviceset="+12V" device=""/>
+<part name="D1" library="diode" deviceset="DIODE-" device="SMB"/>
+<part name="L1" library="inductors" deviceset="DR125" device=""/>
 </parts>
 <sheets>
@@
 <instance part="Q2" gate="G$1" x="154.94" y="-20.32" rot="MR180"/>
 <instance part="Q3" gate="G$1" x="154.94" y="-5.08"/>
+<instance part="U1" gate="A" x="175.26" y="157.48"/>
+<instance part="R1" gate="G$1" x="132.08" y="147.32" rot="R90"/>
+<instance part="R2" gate="G$1" x="157.48" y="111.76" rot="R270"/>
+<instance part="R3" gate="G$1" x="157.48" y="127" rot="R270"/>
+<instance part="C1" gate="G$1" x="132.08" y="134.62"/>
+<instance part="GND6" gate="1" x="154.94" y="142.24"/>
+<instance part="GND7" gate="1" x="157.48" y="101.6"/>
+<instance part="GND8" gate="1" x="132.08" y="124.46"/>
+<instance part="C2" gate="G$1" x="121.92" y="160.02"/>
+<instance part="C3" gate="G$1" x="198.12" y="129.54"/>
+<instance part="GND9" gate="1" x="121.92" y="147.32"/>
+<instance part="GND10" gate="1" x="198.12" y="119.38"/>
+<instance part="P+9" gate="1" x="121.92" y="167.64"/>
+<instance part="D1" gate="G$1" x="198.12" y="147.32" rot="R270"/>
+<instance part="L1" gate="G$1" x="175.26" y="177.8"/>
 </instances>
 <busses>
@@
 <pinref part="X3" gate="-1" pin="1"/>
 <wire x1="43.18" y1="-53.34" x2="48.26" y2="-53.34" width="0.1524" layer="91"/>
+</segment>
+<segment>
+<pinref part="R2" gate="G$1" pin="2"/>
+<pinref part="GND7" gate="1" pin="GND"/>
+<wire x1="157.48" y1="106.68" x2="157.48" y2="104.14" width="0.1524" layer="91"/>
+</segment>
+<segment>
+<pinref part="U1" gate="A" pin="GND_2"/>
+<pinref part="GND6" gate="1" pin="GND"/>
+<wire x1="157.48" y1="149.86" x2="154.94" y2="149.86" width="0.1524" layer="91"/>
+<wire x1="154.94" y1="149.86" x2="154.94" y2="147.32" width="0.1524" layer="91"/>
+<pinref part="U1" gate="A" pin="GND"/>
+<wire x1="154.94" y1="147.32" x2="154.94" y2="144.78" width="0.1524" layer="91"/>
+<wire x1="157.48" y1="147.32" x2="154.94" y2="147.32" width="0.1524" layer="91"/>
+<junction x="154.94" y="147.32"/>
+</segment>
+<segment>
+<pinref part="GND8" gate="1" pin="GND"/>
+<pinref part="C1" gate="G$1" pin="2"/>
+<wire x1="132.08" y1="127" x2="132.08" y2="129.54" width="0.1524" layer="91"/>
+</segment>
+<segment>
+<pinref part="GND9" gate="1" pin="GND"/>
+<pinref part="C2" gate="G$1" pin="-"/>
+<wire x1="121.92" y1="149.86" x2="121.92" y2="154.94" width="0.1524" layer="91"/>
+</segment>
+<segment>
+<pinref part="GND10" gate="1" pin="GND"/>
+<pinref part="C3" gate="G$1" pin="-"/>
+<wire x1="198.12" y1="121.92" x2="198.12" y2="124.46" width="0.1524" layer="91"/>
 </segment>
 </net>
@@
 </segment>
 </net>
+<net name="N$2" class="0">
+<segment>
+<pinref part="R3" gate="G$1" pin="2"/>
+<pinref part="R2" gate="G$1" pin="1"/>
+<wire x1="157.48" y1="121.92" x2="157.48" y2="119.38" width="0.1524" layer="91"/>
+<wire x1="157.48" y1="119.38" x2="157.48" y2="116.84" width="0.1524" layer="91"/>
+<wire x1="157.48" y1="119.38" x2="149.86" y2="119.38" width="0.1524" layer="91"/>
+<wire x1="149.86" y1="119.38" x2="149.86" y2="154.94" width="0.1524" layer="91"/>
+<junction x="157.48" y="119.38"/>
+<pinref part="U1" gate="A" pin="FB"/>
+<wire x1="149.86" y1="154.94" x2="157.48" y2="154.94" width="0.1524" layer="91"/>
+</segment>
+</net>
+<net name="N$3" class="0">
+<segment>
+<pinref part="U1" gate="A" pin="COMP"/>
+<pinref part="R1" gate="G$1" pin="2"/>
+<wire x1="157.48" y1="157.48" x2="132.08" y2="157.48" width="0.1524" layer="91"/>
+<wire x1="132.08" y1="157.48" x2="132.08" y2="152.4" width="0.1524" layer="91"/>
+</segment>
+</net>
+<net name="N$4" class="0">
+<segment>
+<pinref part="R1" gate="G$1" pin="1"/>
+<pinref part="C1" gate="G$1" pin="1"/>
+<wire x1="132.08" y1="142.24" x2="132.08" y2="137.16" width="0.1524" layer="91"/>
+</segment>
+</net>
+<net name="N$8" class="0">
+<segment>
+<pinref part="C3" gate="G$1" pin="+"/>
+<wire x1="198.12" y1="132.08" x2="157.48" y2="132.08" width="0.1524" layer="91"/>
+<pinref part="D1" gate="G$1" pin="C"/>
+<wire x1="198.12" y1="144.78" x2="198.12" y2="132.08" width="0.1524" layer="91"/>
+<junction x="198.12" y="132.08"/>
+</segment>
+</net>
+<net name="+12V" class="0">
+<segment>
+<pinref part="C2" gate="G$1" pin="+"/>
+<pinref part="U1" gate="A" pin="VIN"/>
+<wire x1="121.92" y1="162.56" x2="157.48" y2="162.56" width="0.1524" layer="91"/>
+<pinref part="P+9" gate="1" pin="+12V"/>
+<wire x1="121.92" y1="162.56" x2="121.92" y2="165.1" width="0.1524" layer="91"/>
+<junction x="121.92" y="162.56"/>
+<wire x1="157.48" y1="162.56" x2="157.48" y2="177.8" width="0.1524" layer="91"/>
+<junction x="157.48" y="162.56"/>
+<pinref part="L1" gate="G$1" pin="1"/>
+<wire x1="157.48" y1="177.8" x2="167.64" y2="177.8" width="0.1524" layer="91"/>
+</segment>
+</net>
+<net name="N$7" class="0">
+<segment>
+<pinref part="U1" gate="A" pin="SW"/>
+<pinref part="D1" gate="G$1" pin="A"/>
+<wire x1="193.04" y1="162.56" x2="198.12" y2="162.56" width="0.1524" layer="91"/>
+<wire x1="198.12" y1="162.56" x2="198.12" y2="149.86" width="0.1524" layer="91"/>
+<pinref part="L1" gate="G$1" pin="2"/>
+<wire x1="182.88" y1="177.8" x2="198.12" y2="177.8" width="0.1524" layer="91"/>
+<wire x1="198.12" y1="177.8" x2="198.12" y2="162.56" width="0.1524" layer="91"/>
+<junction x="198.12" y="162.56"/>
+</segment>
+</net>
