File: LED_MagSwitch/MagSwitch.brd (EAGLE design)
At the start: 35 x 30 mm, 16 parts, among them Q1 MMBT2222A, X1 MSTBA2, X2 MSTBA4

Commit message: Magswitch Revision
Parts:
- removed R6: 1k, resistor:M0805
- added D2: DIODE-ZENER8V, RobThePyro:SOD-323
- added Q2: MMBT2222A, SparkFun-DiscreteSemi:SOT23-3
- R4, R5: value 1k -> 4k7
- moved R4 50.0 mm to (-4.90, -12.3), flipped to the top, turned to 0 degrees
- moved R5 49.5 mm to (-4.90, -18.4), flipped to the top
- moved R3 41.7 mm to (-1.80, -6.20), flipped to the top, turned to 0 degrees
Connections:
- new net N$13: Q1.3, Q2.1, R5.1
- net +24V: now also D2.C, X2.3; no longer F1.P$2, R3.1
- net GND: no longer R6.1, X1.1
- net N$1: now also D2.A, R3.1, R4.1; no longer R4.2, R5.1, R6.2, X1.2
- net N$2: now also R4.2; no longer R3.2, R4.1
- net N$3: now also Q1.2, Q2.2, R3.2
- net N$4: now also X1.1; no longer Q1.2
- net N$6: now also F1.P$2, X2.1; no longer F1.P$1, X2.3
- net N$7: now also Q2.3, X1.2; no longer Q1.3
- net OUT-: now also F1.P$1; no longer X2.1
Routing:
- net N$1: track 24.2 -> 0.00 mm
- net +24V: track 32.1 -> 18.2 mm
- net GND: track 27.6 -> 16.3 mm
- net N$7: track 14.8 -> 8.06 mm
- net N$2: track 5.50 -> 0.00 mm
- net N$6: track 4.70 -> 0.00 mm
