File: LED_MagSwitch/MagSwitch.sch (EAGLE design)
At the start: 6 parts, among them X1 MSTBA2, X2 MSTBA4

Commit message: MagSwitch ready to prototype!
Parts:
- added C1: 100nF, resistor:C-USC0805
- added Q1: MMBT2222A, SparkFun-DiscreteSemi:TRANSISTOR_NPNMMBT2222A
- added R2, R3: 10k, resistor:R-US_M0805
- added R4, R5, R6: 1k, resistor:R-US_M0805
- added U$2: DMG4466SSS, RobThePyro:DMG4466SSS
- added U$3: DIODE_TVS_BISM6T30CAY, RobThePyro:DIODE_TVS_BISM6T30CAY
- added U$4: SHROOM5MM, RobThePyro:SHROOM5MM
- D1: value (none) -> DIODE-ZENER15V; device adafruit:DIODESMA -> RobThePyro:DIODE-ZENER15V
- R1: value 10k -> 5k6
- U$1: value NTD5806N -> DMG4466SSS; device RobThePyro:NTD5806N -> RobThePyro:DMG4466SSS
Connections:
- new net N$4: Q1.E, R2.1, U$1.G
- new net N$6: F1.1, X2-3.1
- new net N$7: C1.1, D1.C, Q1.C, R1.2, U$2.G
- net +24V: now also F1.2, R3.1, R5.2, U$3.P$2; no longer X2-3.1
- net GND: now also R6.1, U$2.D, U$3.P$1; no longer U$1.S
- net N$1: now also R4.2, R5.1, R6.2, X1-2.1; no longer D1.A, X2-1.1
- net N$2: now also Q1.B, R3.2, R4.1; no longer R1.2, U$1.G, X1-2.1
- net N$3: now also C1.2, D1.A, R2.2, U$1.S, U$2.S; no longer D1.C, F1.1
- net OUT-: now also X2-1.1; no longer F1.2
Other:
- moved on the sheet: F1, R1, U$1, X1-1, X1-2, X2-1, X2-2
