File: LED_MagSwitch/MagSwitchRev1_2.brd (EAGLE design)
At the start: 35 x 30 mm, 11 parts, among them X1 SWT1, X2 MSTBA4

Commit message: CameraSliderFirmware dev
Parts:
- added R3: 100, resistor:M0805
Connections:
- new net N$3: R3.1, X1.2
- net 15V: now also R3.2; no longer X1.2
Routing:
- net 15V: track 46.2 -> 45.3 mm
Changed lines of the file:
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@@
 <circle x="32" y="27" radius="0.538515625" width="0.3048" layer="16"/>
 <circle x="32" y="12.5" radius="0.565684375" width="0.3048" layer="16"/>
+<dimension x1="0" y1="0" x2="0" y2="30" x3="-4.3" y3="15" textsize="0.0508" layer="16"/>
+<dimension x1="0" y1="30" x2="35" y2="30" x3="17.5" y3="32.7" textsize="0.0508" layer="16"/>
 </plain>
 <attributes>
@@
 <element name="U$1" library="RobThePyro" package="TO252" value="DMN6068LK3" x="13.1" y="25.9" rot="MR270"/>
 <element name="U$2" library="RobThePyro" package="TO252" value="DMN6068LK3" x="22.7" y="17.8" rot="MR90"/>
+<element name="R3" library="resistor" package="M0805" value="100" x="-4.3" y="-6.2"/>
 </elements>
 <signals>
@@
 <contactref element="R2" pad="1"/>
 <contactref element="U$1" pad="1"/>
-<contactref element="X1" pad="2"/>
-<wire x1="31.34" y1="6.88" x2="31.34" y2="7.76" width="0.8128" layer="16"/>
 <wire x1="31.34" y1="7.76" x2="28.5" y2="10.6" width="0.8128" layer="16"/>
 <wire x1="28.5" y1="10.6" x2="28.5" y2="12.9" width="0.8128" layer="16"/>
@@
 <wire x1="22.617" y1="26.3714" x2="22.3756" y2="26.6128" width="0.8128" layer="16"/>
 <wire x1="22.3756" y1="26.6128" x2="20.5472" y2="26.6128" width="0.8128" layer="16"/>
+<contactref element="R3" pad="2"/>
+<wire x1="-3.35" y1="-6.2" x2="17.9" y2="15.52" width="0" layer="19" extent="1-16"/>
 </signal>
 <signal name="N$5">
@@
 <wire x1="26.26" y1="11.0104" x2="26.26" y2="6.88" width="0.8128" layer="16"/>
 </signal>
+<signal name="N$3">
+<contactref element="X1" pad="2"/>
+<contactref element="R3" pad="1"/>
+<wire x1="-5.25" y1="-6.2" x2="31.34" y2="6.88" width="0" layer="19" extent="1-1"/>
+</signal>
 </signals>
