File: MS/MS_Electron_SC/MS_Electron_SC.sch (EAGLE design)
At the start: 2 parts

Commit message: Working on MS electron
Parts:
- added C1, C2, C3, C4: 100nf, OPL_Capacitor:CERAMIC-100NF-50V-10%-X7R(0805)
- added D1: CLEAR-BLUE-0805, OPL_Optoelectronics:SMD-LED-CLEAR-BLUE(0805)
- added D2, D4, D6: MMSD4148-sod123, OPL_Discrete_Semiconductor:SMD-DIODE-100V-200MA(SOD-123)
- added D3, D5, D7: RED-0805, OPL_Optoelectronics:SMD-LED-CLEAR-RED(0805)
- added J1, J2, J3: (no value), SparkFun-Connectors:CONN_03SCREW
- added JP1: JUMPER-SMT_2_NC_TRACE_SILK, SparkFun-Jumpers:JUMPER-SMT_2_NC_TRACE_SILK
- added JP2, JP3: JUMPER-SMT_2_NO_SILK, SparkFun-Jumpers:JUMPER-SMT_2_NO_SILK
- added K1, K2, K3: G5LE, relay:G5LE
- added R1, R10, R5, R6, R7, R8, R9: 1K, OPL_Resistor:SMD-RES-1K-5%-1/8W(0805)
- added R2, R3, R4: 120, OPL_Resistor:SMD-RES-120R-1%-1/8W(0805)
- added U$10, U$6, U$8: MMBT3904LT1G, OPL_Discrete_Semiconductor:SMD-TRANSISTORS-NPN-40V-200MA-MMBT3904LT1G(SOT-23)
- added U$3: MICROSD, adafruit:MICROSD
- added U$4: MCP2551-I/P, Microchip_By_element14_Batch_1:MCP2551-I/P
- added U$5, U$7, U$9: 10K, OPL_Resistor:SMD-RES-10K-1%-1/8W(0805)
- added U1: MAX3485CSA, SparkFun-IC-Comms:RS485SOIC
- added X1, X2, X3: (no value), con-molex-micro-fit-3_0:HEADER_POS2_43650-0200
- U$1: value ELECTRON_WITH_HEADERS -> ELECTRON_WITH_STACKABLE_HEADERS; device Particle-Devices:ELECTRON_WITH_HEADERS -> Particle-Devices:ELECTRON_WITH_STACKABLE_HEADERS
Connections:
- net CANRX renamed CAN1_RX
- net CANTX renamed CAN1_TX
- new net !RE: U$1.B2, U1./RE
- new net +5V: R1.2, U$1.VIN, X3.1
- new net A: JP1.2, U1.A
- new net ACCEL_INT1: U$1.WKP
- new net B: R2.2, U1.B
- new net CAN2_RX: U$1.D2, U$4.RXD
- new net CAN2_TX: U$1.D1, U$4.TXD
- new net CANH1: JP2.1, U$2.CANH, X1.1
- new net CANH2: JP3.1, U$4.CANH, X2.1
- new net CANL1: R3.2, U$2.CANL, X1.2
- new net CANL2: R4.2, U$4.CANL, X2.2
- new net DAC: U$1.DAC
- new net DE: U$1.B1, U1.DE
- new net DI: U$1.B0, U1.DI
- new net GND: C1.1, C2.1, C3.1, C4.1, D1.-, U$1.GND@2, U$1.GND@21, U$10.E, U$2.VSS, U$3.GND, U$3.GND1, U$3.VSS, U$4.VSS, U$5.1, U$6.E, U$7.1, U$8.E, U$9.1, U1.GND, X3.2
- new net GPS_PWR_EN: U$1.D6
- new net GPS_RXD: U$1.TX
- new net GPS_TXD: U$1.RX
- new net MISO: U$1.A4, U$3.DATA_OUT
- new net MISO1: U$1.D3
- new net MOSI: U$1.A5, U$3.DATA_IN
- new net N$1: D1.+, R1.1
- new net N$10: J1.3, K12.S
- new net N$11: D4.+, D5.-, K21.2, U$8.C
- new net N$12: R7.1, U$7.2, U$8.B
- new net N$13: D5.+, R8.2
- new net N$14: J2.2, K22.P
- new net N$15: J2.1, K22.O
- new net N$16: J2.3, K22.S
- new net N$17: D6.+, D7.-, K31.2, U$10.C
- new net N$18: R9.1, U$10.B, U$9.2
- new net N$19: D7.+, R10.2
- new net N$2: JP2.2, R3.1
- new net N$20: J3.2, K32.P
- new net N$21: J3.1, K32.O
- new net N$22: J3.3, K32.S
- new net N$3: JP1.1, R2.1
- new net N$4: JP3.2, R4.1
- new net N$5: R5.1, U$5.2, U$6.B
- new net N$6: D2.+, D3.-, K11.2, U$6.C
- new net N$7: D3.+, R6.2
- new net N$8: J1.2, K12.P
- new net N$9: J1.1, K12.O
- new net RELAY1: R5.2
- new net RELAY2: R7.2
- new net RELAY3: R9.2
- new net RO: U$1.B3, U1.RO
- new net SCK: U$1.A3, U$3.SCLK
- new net SCK1: U$1.D4
- new net SS: U$1.A2, U$3.CS
- new net SS1: U$1.D5
- new net VDD: C1.2, C2.2, C3.2, C4.2, D2.-, D4.-, D6.-, K11.1, K21.1, K31.1, R10.1, R6.1, R8.1, U$1.3V3, U$2.VDD, U$3.VDD, U$4.VDD, U1.VCC
Other:
- moved on the sheet: U$2

Commit message: More MS dev
Parts:
- added C5, C6: 100nf, OPL_Capacitor:CERAMIC-100NF-50V-10%-X7R(0805)
- added D8: MMSD4148-sod123, OPL_Discrete_Semiconductor:SMD-DIODE-100V-200MA(SOD-123)
- added D9: RED-0805, OPL_Optoelectronics:SMD-LED-CLEAR-RED(0805)
- added IC1: MCP23017SO, adafruit:MCP23017SO
- added J4: (no value), SparkFun-Connectors:CONN_03SCREW
- added JP4, JP5, JP6: JUMPER-SMT_3_1-NC_TRACE_SILK, SparkFun-Jumpers:JUMPER-SMT_3_1-NC_TRACE_SILK
- added K4: G5LE, relay:G5LE
- added R11, R12, R13, R14, R15: 1K, OPL_Resistor:SMD-RES-1K-5%-1/8W(0805)
- added U$11: 10K, OPL_Resistor:SMD-RES-10K-1%-1/8W(0805)
- added U$12: MMBT3904LT1G, OPL_Discrete_Semiconductor:SMD-TRANSISTORS-NPN-40V-200MA-MMBT3904LT1G(SOT-23)
- added U2: MCP2515, SparkFun-IC-Comms:MCP2515(MCP2510)SO
- added X4: (no value), con-molex-micro-fit-3_0:HEADER_POS6_43045-0600
Connections:
- new net LEDO1: IC1.GPA4, R13.2
- new net LEDO2: IC1.GPA5, R14.2
- new net LEDO3: IC1.GPA6, R15.2
- new net MOSI1: U$1.D2
- new net N$23: D8.+, D9.-, K41.2, U$12.C
- new net N$24: R11.1, U$11.2, U$12.B
- new net N$25: D9.+, R12.2
- new net N$26: J4.2, K42.P
- new net N$27: J4.1, K42.O
- new net N$28: J4.3, K42.S
- new net N$29: R13.1, X4.1
- new net N$30: R14.1, X4.3
- new net N$31: IC1.A0, JP6.2
- new net N$32: R15.1, X4.5
- new net N$33: IC1.A1, JP4.2
- new net N$34: IC1.A2, JP5.2
- new net RELAY4: IC1.GPA3, R11.2
- new net SCL: IC1.SCL, U$1.D1
- new net SDA: IC1.SDA, U$1.D0
- net +5V: now also C5.2, IC1.!RESET, IC1.VDD, JP4.1, JP5.1, JP6.1
- net CAN2_RX: no longer U$1.D2
- net CAN2_TX: no longer U$1.D1
- net GND: now also C5.1, C6.1, IC1.VSS, JP4.3, JP5.3, JP6.3, U$11.1, U$12.E, X4.2, X4.4, X4.6
- net RELAY1: now also IC1.GPA0
- net RELAY2: now also IC1.GPA1
- net RELAY3: now also IC1.GPA2
- net VDD: now also C6.2, D8.-, K41.1, R12.1

Commit message: Added Isolated CANBUS etc
Parts:
- removed U$2: MCP2551-I/P, Microchip_By_element14_Batch_1:MCP2551-I/P
- removed X2: (no value), con-molex-micro-fit-3_0:HEADER_POS2_43650-0200
- added C10, C11: 560PF 50V, OPL_Capacitor:CERAMIC-390PF-50V-10%-X7R(0402)
- added C12, C13, C14, C7, C8: 100nf, OPL_Capacitor:CERAMIC-100NF-50V-10%-X7R(0805)
- added C9: (no value), OPL_Capacitor:CERAMIC-22UF-16V-10%-X7R(1206)
- added IC2: ISO1050DUB, texas:ISO1050DUB
- added JP7: JUMPER-SMT_3_1-NC_TRACE_SILK, SparkFun-Jumpers:JUMPER-SMT_3_1-NC_TRACE_SILK
- added JP8: JUMPER-SMT_2_NO_SILK, SparkFun-Jumpers:JUMPER-SMT_2_NO_SILK
- added R16, R17: 100, OPL_Resistor:SMD-RES-100R-1%-1/8W(0805)
- added R18: 1M, OPL_Resistor:SMD-RES-1M-1%-1/8W(0805)
- added R19, R20: 4.7k, OPL_Resistor:SMD-RES-4.7K-1%-1/8W(0805)
- added R21: 120, OPL_Resistor:SMD-RES-120R-1%-1/8W(0805)
- added U$14, U$17: 10K, OPL_Resistor:SMD-RES-10K-1%-1/8W(0805)
- added U3: RFB-0505S, SparkFun-IC-Power:RFB-0505S
- added U4, U5: MCP2551, SparkFun-IC-Comms:MCP2551
- added X5, X6: (no value), con-molex-micro-fit-3_0:HEADER_POS3_43650-0300
- added Y1: 16MHZ, OPL_Crystal Oscillator:SMD-RESONATOR-16MHZ-15PF-0.5%-40R(3P-3.2X1.3MM)
- U$4: value MCP2551-I/P -> 10K; device Microchip_By_element14_Batch_1:MCP2551-I/P -> OPL_Resistor:SMD-RES-10K-1%-1/8W(0805)
- X1: device con-molex-micro-fit-3_0:HEADER_POS2_43650-0200 -> con-molex-micro-fit-3_0:HEADER_POS4_43045-0401
Connections:
- new net CAN2_INT: U2>NAME.INT
- new net CAN2_RST: U$14.2, U2>NAME.RESET
- new net GND-ISO: C10.1, C11.1, C8.1, IC2.GND2, JP7.3, U3.VOUT-
- new net INTB: IC1.INTB, U$1.C0
- new net N$35: JP8.2, R21.1
- new net N$36: U$4.2, U5.RS
- new net N$37: C10.2, R17.1
- new net N$38: C11.2, R16.1
- new net N$39: R18.1, U2>NAME.OSC2, Y1.3
- new net N$40: R18.2, U2>NAME.OSC1, Y1.1
- new net N$42: JP7.2, X5.1
- new net N$43: U$17.2, U4.RS
- new net SWT0: IC1.GPB0
- new net SWT1: IC1.GPB1
- new net SWT2: IC1.GPB2
- new net SWT3: IC1.GPB3
- new net VCC-ISO: C8.2, IC2.VCC2, U3.VOUT+
- net +5V: now also C13.2, C14.2, C7.2, C9.2, U3.VIN+, U4.VDD, U5.VDD
- net CAN1_RX: now also IC2.RXD, U5.RXD; no longer U$2.RXD
- net CAN1_TX: now also IC2.TXD, U5.TXD; no longer U$2.TXD
- net CAN2_RX: now also U2>NAME.RXCAN, U4.RXD; no longer U$4.RXD
- net CAN2_TX: now also U2>NAME.TXCAN, U4.TXD; no longer U$4.TXD
- net CANH1: now also IC2.CANH, R16.2, R21.2, R3.2, U5.CANH, X5.2; no longer JP2.1, U$2.CANH, X1.1
- net CANH2: now also R4.2, U4.CANH, X6.2; no longer JP3.1, U$4.CANH, X2.1
- net CANL1: now also IC2.CANL, JP2.1, JP8.1, R17.2, U5.CANL, X5.3; no longer R3.2, U$2.CANL, X1.2
- net CANL2: now also JP3.1, U4.CANL, X6.3; no longer R4.2, U$4.CANL, X2.2
- net GND: now also C12.1, C13.1, C14.1, C7.1, C9.1, IC2.GND1, JP7.1, U$17.1, U$4.1, U2P.VSS, U3.VIN-, U4.VSS, U5.VSS, X6.1, Y1.2; no longer U$2.VSS, U$4.VSS
- net MISO1: now also U2>NAME.SO
- net MOSI1: now also U2>NAME.SI
- net SCK1: now also U2>NAME.SCK
- net SCL: now also R19.1
- net SDA: now also R20.1
- net SS1: now also U2>NAME.CS
- net VDD: now also C12.2, IC2.VCC1, R19.2, R20.2, U$14.1, U2P.VDD, U4.VREF, U5.VREF; no longer U$2.VDD, U$4.VDD
Other:
- moved on the sheet: C1, C2, C3, C6, JP2, JP3, R3, R4, U2

Commit message: Added datasheets etc
Parts:
- added C15, C16: 560PF 50V, OPL_Capacitor:CERAMIC-390PF-50V-10%-X7R(0402)
- added C17, C18, C19, C20, C23, C24: 10nf, OPL_Capacitor:CERAMIC-10NF-50V-5%-X7R(0805)
- added C21: 100nf, OPL_Capacitor:CERAMIC-100NF-50V-10%-X7R(0805)
- added C22: 10uf, OPL_Capacitor:TANTALUM-SMD-10UF-10V-10%(AVX-A)
- added D10, D11: PESD1CAN, diode:PESD1CAN
- added D12, D13, D14, D15, D16: 5V-225MW, OPL_Circuit_Protection:SMD-DIODE-TVS-5V-225MW(SOT-23)
- added JP9: JUMPER-SMT_3_1-NC_TRACE_SILK, SparkFun-Jumpers:JUMPER-SMT_3_1-NC_TRACE_SILK
- added R22, R23: 100, OPL_Resistor:SMD-RES-100R-1%-1/8W(0805)
- added R24, R25, R26, R27: 1K, OPL_Resistor:SMD-RES-1K-5%-1/8W(0805)
- added R28, R29, R30, R31: 100k, OPL_Resistor:SMD-RES-100K-1%-1/8W(0805)
- added R32, R33: 15k, OPL_Resistor:SMD-RES-15K-5%-1/8W(0805)
- added R34, R35: 2k, OPL_Resistor:SMD-RES-2K-1%-1/8W(0805)
- added U6: MCP4725, SparkFun-IC-Conversion:MCP4725SOT-23
- added X2: (no value), con-molex-micro-fit-3_0:HEADER_POS3_43650-0300
- added X7, X8: (no value), con-molex-micro-fit-3_0:HEADER_POS2_43650-0200
Connections:
- new net 5VDAC: D16.3, U6.VOUT, X2.2
- new net ADC0: C24.1, R32.1, R35.2, U$1.A0
- new net ADC1: C23.1, R33.1, R34.2, U$1.A1
- new net N$41: C10.1, C11.1, D10.3, JP7.2, X5.1
- new net N$44: C16.2, R22.1
- new net N$45: R24.1, X1.1
- new net N$46: R25.1, X1.2
- new net N$47: R26.1, X1.3
- new net N$48: R27.1, X1.4
- new net N$49: JP9.2, U6.AO
- new net N$50: R33.2, X8.1
- new net N$51: R32.2, X7.1
- net +5V: now also C21.2, C22.-, D12.1, D13.1, D14.1, D15.1, D16.1, JP9.1, R19.2, R20.2, R28.2, R29.2, R30.2, R31.2, U6.VDD, X2.1
- net CANH1: now also D10.1
- net CANH2: now also D11.1, R22.2
- net CANL1: now also D10.2
- net CANL2: now also D11.2, R23.2
- net GND: now also C15.1, C16.1, C17.2, C18.2, C19.2, C20.2, C21.1, C22.+, C23.2, C24.2, D11.3, D12.2, D13.2, D14.2, D15.2, D16.2, JP9.3, R34.1, R35.1, U6.VSS, X2.3, X7.2, X8.2
- net GND-ISO: no longer C10.1, C11.1
- net N$42: now also C15.2, R23.1; no longer JP7.2, X5.1
- net SCL: now also U6.SCL
- net SDA: now also U6.SDA
- net SWT0: now also C20.1, D15.3, R24.2, R31.1
- net SWT1: now also C19.1, D14.3, R25.2, R30.1
- net SWT2: now also C18.1, D13.3, R26.2, R29.1
- net SWT3: now also C17.1, D12.3, R27.2, R28.1
- net VDD: no longer R19.2, R20.2
Other:
- moved on the sheet: C10, C11, R16, R17, X1, X5, X6

Commit message: Neatened Schematic
Connections:
- net N$10: now also J1.1; no longer J1.3
- net N$15: now also J2.3; no longer J2.1
- net N$16: now also J2.1; no longer J2.3
- net N$21: now also J3.3; no longer J3.1
- net N$22: now also J3.1; no longer J3.3
- net N$27: now also J4.3; no longer J4.1
- net N$28: now also J4.1; no longer J4.3
- net N$9: now also J1.3; no longer J1.1
Other:
- note added: "CAN1"
- note added: "CAN2"
- note added: "I2C DAC"
- note added: "I2C IO"
- note added: "IO"
- note added: "Optional"
- note added: "Particle Electron"
- note added: "Power"
- note added: "RS485"
- note added: "mSD CARD"
- moved on the sheet: C1, C10, C11, C12, C13, C14, C15, C16, C17, C18, C19, C2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

Commit message: Layout started
Parts:
- removed JP8: JUMPER-SMT_2_NO_SILK, SparkFun-Jumpers:JUMPER-SMT_2_NO_SILK
- removed R21: 120, OPL_Resistor:SMD-RES-120R-1%-1/8W(0805)
- removed U$3: MICROSD, adafruit:MICROSD
- added CT1, CT2, CT3: 220UF, OPL_Capacitor:ALUMINUM-SMD-220UF-16V(D6.3-H7.7MM)
- added F1, F2: (no value), adafruit:PTCFUSE-1812
- added JP10, JP11: (no value), adafruit:PINHD-1X18-BIG
- added SD1: ST-TF-003A, OPL_Connector:MICRO-SD-CARD-SOCKET-9P(ST-TF-003A)
- added X9: (no value), con-molex-micro-fit-3_0:HEADER_POS6_43045-0600
- U$1: value ELECTRON_WITH_STACKABLE_HEADERS -> ELECTRON_WITH_HEADERS; device Particle-Devices:ELECTRON_WITH_STACKABLE_HEADERS -> Particle-Devices:ELECTRON_WITH_HEADERS
Connections:
- new net 5V: X9.5
- new net GPS_PPS: X9.6
- new net N$52: JP11.17, U$1.!RST
- new net N$53: JP11.16, U$1.VBAT
- new net N$54: F1.1, JP10.1, U$1.VIN
- net +5V: now also CT1.+, CT2.+, CT3.+, D2.-, D4.-, D6.-, D8.-, F1.2, K11.1, K21.1, K31.1, K41.1, R10.1, R12.1, R6.1, R8.1; no longer U$1.VIN
- net ACCEL_INT1: now also JP10.5
- net CANH1: no longer R21.2
- net CANL1: no longer JP8.1
- net GND: now also CT1.-, CT2.-, CT3.-, JP10.2, JP11.15, SD1.G1, SD1.G2, SD1.G3, SD1.G4, SD1.VSS, X4.1, X4.3, X9.2; no longer U$3.GND, U$3.GND1, U$3.VSS, X4.4, X4.6
- net GPS_PWR_EN: now also JP11.13, X9.1
- net GPS_RXD: now also JP10.3, X9.3
- net GPS_TXD: now also JP10.4, X9.4
- net LEDO1: now also R15.2; no longer R13.2
- net LEDO3: now also R13.2; no longer R15.2
- net MISO: now also JP10.8, SD1.DO; no longer U$3.DATA_OUT
- net MOSI: now also JP10.7, SD1.DI; no longer U$3.DATA_IN
- net N$29: now also R14.1, X4.5; no longer R13.1, X4.1
- net N$30: now also R13.1, X4.4; no longer R14.1, X4.3
- net N$32: now also X4.6; no longer X4.5
- net N$35: now also F2.1, JP11.18, U$1.3V3; no longer JP8.2, R21.1
- net SCK: now also JP10.9, SD1.SCLK; no longer U$3.SCLK
- net SCL: now also JP11.8
- net SDA: now also JP11.7
- net SS: now also SD1.CS; no longer U$3.CS
- net VDD: now also F2.2, SD1.VDD; no longer D2.-, D4.-, D6.-, D8.-, K11.1, K21.1, K31.1, K41.1, R10.1, R12.1, R6.1, R8.1, U$1.3V3, U$3.VDD
Other:
- moved on the sheet: C1, R13, R14, R15

Commit message: Layout Almost Done
Parts:
- removed CT3: 220UF, OPL_Capacitor:ALUMINUM-SMD-220UF-16V(D6.3-H7.7MM)
- added D17: (no value), adafruit:DIODESMA
- added F3, F4: (no value), adafruit:PTCFUSE-1812
- added R21: 4k7, OPL_Resistor:SMD-RES-4.7K-1%-1/8W(0805)
- added X10: (no value), con-molex-micro-fit-3_0:HEADER_POS3_43650-0300
- added X11: (no value), con-molex-micro-fit-3_0:HEADER_POS4_43045-0401
- C10, C11, C15, C16: value 560PF 50V -> 560pf; device OPL_Capacitor:CERAMIC-390PF-50V-10%-X7R(0402) -> OPL_Capacitor:CERAMIC-10NF-50V-5%-X7R(0805)
Connections:
- removed net 5V: X9.5
- removed net N$48 (its old number): R27.1, X1.4
- new net 1WIRE: JP11.4, R21.1, U$1.C3, X10.2
- new net N$47: R25.1, X1.4
- new net N$55: D17.A, X3.1
- new net N$56: D17.C, F3.1
- new net N$60: F4.2, X11.1
- net +5V: now also F3.2, F4.1, R21.2, X10.1, X9.5; no longer CT3.+, X3.1
- net A: now also X11.3
- net ADC0: now also JP10.12
- net ADC1: now also JP10.11
- net B: now also X11.4
- net CAN2_INT: now also U$1.C1
- net GND: now also X10.3, X11.2; no longer CT3.-
- net LEDO1: now also R13.2; no longer R15.2
- net LEDO3: now also R15.2; no longer R13.2
- net N$37: now also C11.2; no longer C10.2
- net N$38: now also C10.2; no longer C11.2
- net N$42: now also C16.2; no longer C15.2
- net N$44: now also C15.2; no longer C16.2
- net N$45: now also X1.2; no longer X1.1
- net N$46: now also R27.1, X1.1; no longer R25.1, X1.2
Other:
- moved on the sheet: C10, C11, C15, C16
