File: MS/MS_Electron_SC/MS_Electron_SC.sch (EAGLE design)
At the start: 136 parts, among them IC1 MCP23017SO, IC2 ISO1050DUB, K1 G5LE, K2 G5LE, K3 G5LE, K4 G5LE, U1 MAX3485CSA, U2 MCP2515, U3 RFB-0505S, U4 MCP2551, U5 MCP2551, U6 MCP4725, Y1 16MHZ

Commit message: tweaks
Connections:
- net N$31 renamed ADR0
- net N$33 renamed ADR1
- net N$34 renamed ADR2
Changed lines of the file:
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@@
 </segment>
 </net>
-<net name="N$31" class="0">
+<net name="ADR0" class="0">
 <segment>
 <pinref part="IC1" gate="G$1" pin="A0"/>
@@
 <wire x1="309.88" y1="198.12" x2="266.7" y2="198.12" width="0.1524" layer="91"/>
 <wire x1="266.7" y1="198.12" x2="266.7" y2="193.04" width="0.1524" layer="91"/>
+<label x="266.7" y="195.58" size="1.778" layer="95"/>
 </segment>
 </net>
-<net name="N$33" class="0">
+<net name="ADR1" class="0">
 <segment>
 <pinref part="IC1" gate="G$1" pin="A1"/>
@@
 <wire x1="309.88" y1="195.58" x2="281.94" y2="195.58" width="0.1524" layer="91"/>
 <wire x1="281.94" y1="195.58" x2="281.94" y2="185.42" width="0.1524" layer="91"/>
+<label x="281.94" y="193.04" size="1.778" layer="95"/>
 </segment>
 </net>
-<net name="N$34" class="0">
+<net name="ADR2" class="0">
 <segment>
 <pinref part="IC1" gate="G$1" pin="A2"/>
@@
 <wire x1="309.88" y1="193.04" x2="297.18" y2="193.04" width="0.1524" layer="91"/>
 <wire x1="297.18" y1="193.04" x2="297.18" y2="177.8" width="0.1524" layer="91"/>
+<label x="297.18" y="190.5" size="1.778" layer="95"/>
 </segment>
 </net>
